Commit message: Modified readme and xacro

File: src/my_pckg/meshes/turtlebot3_burger_michael.urdf.xacro (robot description, xacro)
@@ -142,5 +142,5 @@
   <link name="head_link">
     <visual>
-      <origin xyz="0.02 -0.15 0" rpy="0 0 1.57"/> <!-- Adjust xyz and rpy as needed -->
+      <origin xyz="0.02 -0.05 0.2" rpy="0 0 1.57"/> <!-- Adjust xyz and rpy as needed -->
       <geometry>
         <mesh filename="package://my_pckg/meshes/ZombieHunterHead_v4_90k.stl" scale="0.001 0.001 0.001"/>
@@ -151,5 +151,5 @@
     <parent link="base_link"/> <!-- Assuming you are attaching to base_link -->
     <child link="head_link"/>
-    <origin xyz="0.02 -0.15 0" rpy="0 0 1.57"/> <!-- Same as in head_link origin -->
+    <origin xyz="0 0 0" rpy="0 0 0"/> <!-- Same as in head_link origin -->
   </joint>
 </robot>
